File: pcb_project/Power.kicad_sch (KiCad schematic)
At the start: 53 parts, among them IC1 TPS54325PWPR, IC2 TPS54294PWPR, J10 M20-9990246, J11 M20-9990246, J12 M20-9990246, J5 USB_B_Micro, J9 M20-9990246, Q3 2N3904, Q4 2N3904

Commit message: Add new LED curcuits to layout
Parts:
- D5, D6, D7, D8: footprint LTST-C190KRKT:LEDC1608X35N -> Project_Footprints:LEDC1608X35N
- R52, R88, R89, R92, R93, R94, R95, R96: footprint (none) -> Resistor_SMD:R_0805_2012Metric_Pad1.20x1.40mm_HandSolder
Changed lines of the file:
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@@
 			)
 		)
-		(property "Footprint" "LTST-C190KRKT:LEDC1608X35N"
+		(property "Footprint" "Project_Footprints:LEDC1608X35N"
 			(at 245.11 133.35 0)
 			(effects
@@
 			)
 		)
-		(property "Footprint" ""
+		(property "Footprint" "Resistor_SMD:R_0805_2012Metric_Pad1.20x1.40mm_HandSolder"
 			(at 243.332 119.38 90)
 			(effects
@@
 			)
 		)
-		(property "Footprint" ""
+		(property "Footprint" "Resistor_SMD:R_0805_2012Metric_Pad1.20x1.40mm_HandSolder"
 			(at 226.822 43.18 90)
 			(effects
@@
 			)
 		)
-		(property "Footprint" ""
+		(property "Footprint" "Resistor_SMD:R_0805_2012Metric_Pad1.20x1.40mm_HandSolder"
 			(at 230.632 109.22 90)
 			(effects
@@
 			)
 		)
-		(property "Footprint" "LTST-C190KRKT:LEDC1608X35N"
+		(property "Footprint" "Project_Footprints:LEDC1608X35N"
 			(at 220.98 41.91 0)
 			(effects
@@
 			)
 		)
-		(property "Footprint" ""
+		(property "Footprint" "Resistor_SMD:R_0805_2012Metric_Pad1.20x1.40mm_HandSolder"
 			(at 226.568 121.92 90)
 			(effects
@@
 			)
 		)
-		(property "Footprint" ""
+		(property "Footprint" "Resistor_SMD:R_0805_2012Metric_Pad1.20x1.40mm_HandSolder"
 			(at 222.758 55.88 90)
 			(effects
@@
 			)
 		)
-		(property "Footprint" "LTST-C190KRKT:LEDC1608X35N"
+		(property "Footprint" "Project_Footprints:LEDC1608X35N"
 			(at 241.3 31.75 0)
 			(effects
@@
 			)
 		)
-		(property "Footprint" ""
+		(property "Footprint" "Resistor_SMD:R_0805_2012Metric_Pad1.20x1.40mm_HandSolder"
 			(at 226.568 143.51 90)
 			(effects
@@
 			)
 		)
-		(property "Footprint" ""
+		(property "Footprint" "Resistor_SMD:R_0805_2012Metric_Pad1.20x1.40mm_HandSolder"
 			(at 226.822 21.59 90)
 			(effects
@@
 			)
 		)
-		(property "Footprint" "LTST-C190KRKT:LEDC1608X35N"
+		(property "Footprint" "Project_Footprints:LEDC1608X35N"
 			(at 232.41 123.19 0)
 			(effects
@@
 			)
 		)
-		(property "Footprint" ""
+		(property "Footprint" "Resistor_SMD:R_0805_2012Metric_Pad1.20x1.40mm_HandSolder"
 			(at 239.522 45.72 90)
 			(effects

Commit message: LED PWR PCB circuit. Watch the head of the ship!
Parts:
- Q3, Q4: value 2N3904 -> MMBT3904LT1G; footprint Package_TO_SOT_THT:TO-92_Inline -> Project_Footprints:SOT95P240X111-3N; symbol Transistor_BJT:2N3904 -> MMBT3904LT1G:MMBT3904LT1G; MANUFACTURER (none) -> ON Semiconductor
Connections:
- net GND: now also Q3.2 (E), Q4.2 (E); no longer Q3.1 (E), Q4.1 (E)
- net at R95.2, R96.1: now also Q4.1 (B); no longer Q4.2 (B)
- net at R92.1, R93.2: now also Q3.1 (B); no longer Q3.2 (B)
Changed lines of the file:
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@@
 	)
 	(junction
+		(at 224.79 138.43)
+		(diameter 0)
+		(color 0 0 0 0)
+	)
+	(junction
 		(at 193.04 48.26)
 		(diameter 0)
@@
 	)
 	(junction
+		(at 228.6 26.67)
+		(diameter 0)
+		(color 0 0 0 0)
+	)
+	(junction
 		(at 105.41 69.85)
 		(diameter 0)
@@
 	)
 	(junction
-		(at 228.6 29.21)
-		(diameter 0)
-		(color 0 0 0 0)
-	)
-	(junction
 		(at 128.27 144.78)
 		(diameter 0)
@@
 	)
 	(junction
-		(at 224.79 135.89)
-		(diameter 0)
-		(color 0 0 0 0)
-	)
-	(junction
 		(at 185.42 144.78)
 		(diameter 0)
@@
 	(wire
 		(pts
-			(xy 228.6 29.21) (xy 228.6 39.37)
+			(xy 228.6 26.67) (xy 228.6 39.37)
 		)
 		(stroke
@@
 	(wire
 		(pts
+			(xy 224.79 125.73) (xy 224.79 138.43)
+		)
+		(stroke
+			(width 0)
+			(type default)
+		)
+	)
+	(wire
+		(pts
 			(xy 50.8 35.56) (xy 50.8 39.37)
 		)
@@
 	(wire
 		(pts
-			(xy 224.79 135.89) (xy 224.79 125.73)
-		)
-		(stroke
-			(width 0)
-			(type default)
-		)
-	)
-	(wire
-		(pts
 			(xy 105.41 35.56) (xy 113.03 35.56)
 		)
@@
 	(wire
 		(pts
-			(xy 228.6 25.4) (xy 228.6 29.21)
+			(xy 228.6 25.4) (xy 228.6 26.67)
 		)
 		(stroke
@@
 	(wire
 		(pts
-			(xy 224.79 139.7) (xy 224.79 135.89)
+			(xy 224.79 139.7) (xy 224.79 138.43)
 		)
 		(stroke
@@
 	)
 	(symbol
-		(lib_id "Transistor_BJT:2N3904")
-		(at 229.87 135.89 0)
+		(lib_id "MMBT3904LT1G:MMBT3904LT1G")
+		(at 229.87 138.43 0)
 		(unit 1)
 		(exclude_from_sim no)
@@
 		(fields_autoplaced yes)
 		(property "Reference" "Q4"
-			(at 234.95 134.6199 0)
+			(at 233.68 137.1599 0)
 			(effects
 				(font
@@
 			)
 		)
-		(property "Value" "2N3904"
-			(at 234.95 137.1599 0)
+		(property "Value" "MMBT3904LT1G"
+			(at 233.68 139.6999 0)
 			(effects
 				(font
@@
 			)
 		)
-		(property "Footprint" "Package_TO_SOT_THT:TO-92_Inline"
-			(at 234.95 137.795 0)
+		(property "Footprint" "Project_Footprints:SOT95P240X111-3N"
+			(at 229.87 138.43 0)
 			(effects
 				(font
 					(size 1.27 1.27)
-					(italic yes)
 				)
-				(justify left)
+				(justify bottom)
 				(hide yes)
 			)
 		)
 		(property "Datasheet" "https://www.onsemi.com/pub/Collateral/2N3903-D.PDF"
-			(at 229.87 135.89 0)
+			(at 229.87 138.43 0)
 			(effects
 				(font
 					(size 1.27 1.27)
 				)
-				(justify left)
 				(hide yes)
 			)
 		)
 		(property "Description" "0.2A Ic, 40V Vce, Small Signal NPN Transistor, TO-92"
-			(at 229.87 135.89 0)
+			(at 229.87 138.43 0)
 			(effects
 				(font
@@
 		)
 		(property "Sim.Pins" ""
-			(at 229.87 135.89 0)
+			(at 229.87 138.43 0)
+			(effects
+				(font
+					(size 1.27 1.27)
+				)
+				(hide yes)
+			)
+		)
+		(property "MANUFACTURER" "ON Semiconductor"
+			(at 229.87 138.43 0)
 			(effects
 				(font
 					(size 1.27 1.27)
 				)
+				(justify bottom)
 				(hide yes)
 			)
@@
 	(symbol
 		(lib_id "power:GND")
-		(at 220.98 24.13 180)
+		(at 220.98 19.05 180)
 		(unit 1)
 		(exclude_from_sim no)
@@
 		(fields_autoplaced yes)
 		(property "Reference" "#PWR0141"
-			(at 220.98 17.78 0)
+			(at 220.98 12.7 0)
 			(effects
 				(font
@@
 		)
 		(property "Value" "GND"
-			(at 220.98 19.05 0)
+			(at 220.98 13.97 0)
 			(effects
 				(font
@@
 		)
 		(property "Footprint" ""
-			(at 220.98 24.13 0)
+			(at 220.98 19.05 0)
 			(effects
 				(font
@@
 		)
 		(property "Datasheet" ""
-			(at 220.98 24.13 0)
+			(at 220.98 19.05 0)
 			(effects
 				(font
@@
 		)
 		(property "Description" "Power symbol creates a global label with name \"GND\" , ground"
-			(at 220.98 24.13 0)
+			(at 220.98 19.05 0)
 			(effects
 				(font
@@
 	)
 	(symbol
-		(lib_id "Transistor_BJT:2N3904")
-		(at 223.52 29.21 180)
+		(lib_id "MMBT3904LT1G:MMBT3904LT1G")
+		(at 223.52 26.67 180)
 		(unit 1)
 		(exclude_from_sim no)
@@
 		(fields_autoplaced yes)
 		(property "Reference" "Q3"
-			(at 218.44 30.4801 0)
+			(at 219.71 25.3999 0)
 			(effects
 				(font
@@
 			)
 		)
-		(property "Value" "2N3904"
-			(at 218.44 27.9401 0)
+		(property "Value" "MMBT3904LT1G"
+			(at 219.71 27.9399 0)
 			(effects
 				(font
@@
 			)
 		)
-		(property "Footprint" "Package_TO_SOT_THT:TO-92_Inline"
-			(at 218.44 27.305 0)
+		(property "Footprint" "Project_Footprints:SOT95P240X111-3N"
+			(at 223.52 26.67 0)
 			(effects
 				(font
 					(size 1.27 1.27)
-					(italic yes)
 				)
-				(justify left)
+				(justify bottom)
 				(hide yes)
 			)
 		)
 		(property "Datasheet" "https://www.onsemi.com/pub/Collateral/2N3903-D.PDF"
-			(at 223.52 29.21 0)
+			(at 223.52 26.67 0)
 			(effects
 				(font
 					(size 1.27 1.27)
 				)
-				(justify left)
 				(hide yes)
 			)
 		)
 		(property "Description" "0.2A Ic, 40V Vce, Small Signal NPN Transistor, TO-92"
-			(at 223.52 29.21 0)
+			(at 223.52 26.67 0)
 			(effects
 				(font
@@
 		)
 		(property "Sim.Pins" ""
-			(at 223.52 29.21 0)
+			(at 223.52 26.67 0)
 			(effects
 				(font
@@
 			)
 		)
+		(property "MANUFACTURER" "ON Semiconductor"
+			(at 223.52 26.67 0)
+			(effects
+				(font
+					(size 1.27 1.27)
+				)
+				(justify bottom)
+				(hide yes)
+			)
+		)
 		(pin "1"
 		)
@@
 	(symbol
 		(lib_id "power:GND")
-		(at 232.41 140.97 0)
+		(at 232.41 146.05 0)
 		(unit 1)
 		(exclude_from_sim no)
@@
 		(fields_autoplaced yes)
 		(property "Reference" "#PWR0142"
-			(at 232.41 147.32 0)
+			(at 232.41 152.4 0)
 			(effects
 				(font
@@
 		)
 		(property "Value" "GND"
-			(at 232.41 146.05 0)
+			(at 232.41 151.13 0)
 			(effects
 				(font
@@
 		)
 		(property "Footprint" ""
-			(at 232.41 140.97 0)
+			(at 232.41 146.05 0)
 			(effects
 				(font
@@
 		)
 		(property "Datasheet" ""
-			(at 232.41 140.97 0)
+			(at 232.41 146.05 0)
 			(effects
 				(font
@@
 		)
 		(property "Description" "Power symbol creates a global label with name \"GND\" , ground"
-			(at 232.41 140.97 0)
+			(at 232.41 146.05 0)
 			(effects
 				(font
